Commit message: AUTO STUFF

File: 30_ros2_ws/src/guardian_description/urdf/guardian.urdf.xacro (robot description, xacro)
@@ -1,27 +1,103 @@
 <?xml version="1.0"?>
-<!-- GUARDIAN URDF/xacro stub -->
-<!-- Owner: Phillipp -->
-<!-- TODO: fill in robot geometry after physical chassis is built -->
-<!-- Measure actual dimensions and update robot_params.yaml to match -->
 <robot name="guardian" xmlns:xacro="http://www.ros.org/wiki/xacro">
-  <!-- TODO: define material properties -->
-  <!-- base_link — center of chassis at ground level -->
+  <!-- ── Materials ─────────────────────────────────────────────────────────── -->
+  <material name="dark_grey">
+    <color rgba="0.2 0.2 0.2 1.0"/>
+  </material>
+  <material name="blue">
+    <color rgba="0.1 0.4 0.8 1.0"/>
+  </material>
+  <material name="red">
+    <color rgba="0.8 0.1 0.1 1.0"/>
+  </material>
+  <!-- ── Chassis (base_link centre = ground level) ─────────────────────────── -->
+  <!--  Physical size: 231.2 mm × 200 mm × 100 mm                               -->
   <link name="base_link">
-    <!-- TODO: add visual and collision geometry -->
+    <visual>
+      <origin xyz="0 0 0.05" rpy="0 0 0"/>
+      <geometry>
+        <box size="0.2312 0.200 0.100"/>
+      </geometry>
+      <material name="dark_grey"/>
+    </visual>
+    <collision>
+      <origin xyz="0 0 0.05" rpy="0 0 0"/>
+      <geometry>
+        <box size="0.2312 0.200 0.100"/>
+      </geometry>
+    </collision>
     <inertial>
-      <!-- TODO: add inertia from CAD model -->
-      <mass value="5.0"/>
-      <origin xyz="0 0 0.1" rpy="0 0 0"/>
-      <inertia ixx="0.1" ixy="0" ixz="0"
-               iyy="0.1" iyz="0"
-               izz="0.1"/>
+      <origin xyz="0 0 0.05" rpy="0 0 0"/>
+      <mass value="4.0"/>
+      <!-- box inertia: m/12*(h²+d²) etc. for 0.2312×0.200×0.100, m=4 kg -->
+      <inertia ixx="0.01517" ixy="0" ixz="0"
+               iyy="0.02250" iyz="0"
+               izz="0.03118"/>
     </inertial>
   </link>
-  <!-- TODO: add wheel links (FL, FR, BL, BR) -->
-  <!-- TODO: add wheel joints with continuous type -->
-  <!-- TODO: add Intel RealSense T265 link and joint -->
-  <!-- T265 frame_id must match ekf_params.yaml odom1 source -->
-  <!-- TODO: add Scanse Sweep LIDAR link and joint -->
-  <!-- LIDAR frame_id must match LaserScan header in lidar_republisher_node -->
-  <!-- TODO: add left and right arm base links and joints -->
+  <!-- ── Wheels (continuous joints, visual only) ───────────────────────────── -->
+  <!-- wheel radius ~50 mm assumed; adjust if different -->
+  <xacro:macro name="wheel" params="name x y">
+    <link name="${name}_wheel">
+      <visual>
+        <origin xyz="0 0 0" rpy="1.5708 0 0"/>
+        <geometry>
+          <cylinder radius="0.05" length="0.04"/>
+        </geometry>
+        <material name="blue"/>
+      </visual>
+      <collision>
+        <origin xyz="0 0 0" rpy="1.5708 0 0"/>
+        <geometry>
+          <cylinder radius="0.05" length="0.04"/>
+        </geometry>
+      </collision>
+      <inertial>
+        <mass value="0.3"/>
+        <inertia ixx="0.000375" ixy="0" ixz="0"
+                 iyy="0.000375" iyz="0"
+                 izz="0.000375"/>
+      </inertial>
+    </link>
+    <joint name="${name}_wheel_joint" type="continuous">
+      <parent link="base_link"/>
+      <child  link="${name}_wheel"/>
+      <origin xyz="${x} ${y} 0" rpy="0 0 0"/>
+      <axis xyz="0 1 0"/>
+    </joint>
+  </xacro:macro>
+  <xacro:wheel name="front_left"  x=" 0.0856"  y=" 0.120"/>
+  <xacro:wheel name="front_right" x=" 0.0856"  y="-0.120"/>
+  <xacro:wheel name="rear_left"   x="-0.0856"  y=" 0.120"/>
+  <xacro:wheel name="rear_right"  x="-0.0856"  y="-0.120"/>
+  <!-- ── Scanse Sweep LIDAR ─────────────────────────────────────────────────── -->
+  <!--  Mounted middle-front at top surface:                                      -->
+  <!--    x = +0.1156 m (front half), y = 0 (centre), z = 0.100 m (top surface)  -->
+  <link name="laser">
+    <visual>
+      <origin xyz="0 0 0.015" rpy="0 0 0"/>
+      <geometry>
+        <cylinder radius="0.04" length="0.03"/>
+      </geometry>
+      <material name="red"/>
+    </visual>
+    <collision>
+      <origin xyz="0 0 0.015" rpy="0 0 0"/>
+      <geometry>
+        <cylinder radius="0.04" length="0.03"/>
+      </geometry>
+    </collision>
+    <inertial>
+      <mass value="0.1"/>
+      <inertia ixx="0.0001" ixy="0" ixz="0"
+               iyy="0.0001" iyz="0"
+               izz="0.0001"/>
+    </inertial>
+  </link>
+  <joint name="laser_joint" type="fixed">
+    <parent link="base_link"/>
+    <child  link="laser"/>
+    <!-- front edge centre, top surface of chassis -->
+    <origin xyz="0.1156 0.0 0.100" rpy="0 0 0"/>
+  </joint>
 </robot>
